File: usbPaddleKicad/usbPaddleKicad.kicad_pcb (KiCad board)
At the start: 0 parts

Commit message: pcb layout first pass, not fully routed
Parts:
- added C1: .1µF, Capacitor_THT:C_Disc_D3.8mm_W2.6mm_P2.50mm, F.Cu at (122.6, 76.0)
- added C2: .1µF, Capacitor_THT:C_Disc_D3.8mm_W2.6mm_P2.50mm, F.Cu at (122.6, 72.0)
- added C3: .1µF, Capacitor_THT:C_Disc_D3.8mm_W2.6mm_P2.50mm, F.Cu at (122.6, 68.0)
- added C4: .1µF, Capacitor_THT:C_Disc_D3.8mm_W2.6mm_P2.50mm, F.Cu at (122.6, 64.0)
- added R1: 10kΩ, Resistor_THT:R_Axial_DIN0309_L9.0mm_D3.2mm_P12.70mm_Horizontal, F.Cu at (169.0, 59.0)
- added R2: 10kΩ, Resistor_THT:R_Axial_DIN0309_L9.0mm_D3.2mm_P12.70mm_Horizontal, F.Cu at (169.3, 77.0)
- added R3: 10kΩ, Resistor_THT:R_Axial_DIN0309_L9.0mm_D3.2mm_P12.70mm_Horizontal, F.Cu at (169.3, 71.0)
- added R4: 10kΩ, Resistor_THT:R_Axial_DIN0309_L9.0mm_D3.2mm_P12.70mm_Horizontal, F.Cu at (169.3, 65.0)
- added U1: RP2040-ZERO, RP2040-ZERO:MODULE_RP2040-ZERO, F.Cu at (136.6, 68.0)
- added U2: RJ116P4C, RJ116P4C:RJ6P4C_GLX-N-64M, F.Cu at (109.6, 91.7)
- added U3: RJ116P4C, RJ116P4C:RJ6P4C_GLX-N-64M, F.Cu at (127.6, 91.7)
- added U4: RJ116P4C, RJ116P4C:RJ6P4C_GLX-N-64M, F.Cu at (145.6, 91.7)
- added U5: RJ116P4C, RJ116P4C:RJ6P4C_GLX-N-64M, F.Cu at (163.6, 91.7)
Routing:
- net VCC: track 0.00 -> 63.0 mm
- net Net-(U1-GP7): track 0.00 -> 14.2 mm
- net Net-(U1-GP2): track 0.00 -> 13.2 mm
- net Net-(U1-GP8): track 0.00 -> 12.8 mm
- net Net-(U1-GP1): track 0.00 -> 12.6 mm
- net Net-(U1-GP26): track 0.00 -> 5.09 mm
- net Net-(U1-GP29): track 0.00 -> 4.48 mm
- net Net-(U1-GP27): track 0.00 -> 4.48 mm
- net Net-(U1-GP28): track 0.00 -> 3.88 mm
- added copper zone on B.Cu, net GND
- added copper zone on F.Cu, net GND
Other:
- board outline added: 90 x 51 mm
- copper layers 0 -> 2
