File: usbPaddleSingleKicad/usbPaddleSingleKicad.kicad_sch (KiCad schematic)
At the start: 5 parts, among them U1 RP2040-ZERO

Commit message: new single paddle pcb
Parts:
- added J1: Conn_01x02_Pin, Connector_PinHeader_2.54mm:PinHeader_1x02_P2.54mm_Vertical, symbol Connector:Conn_01x02_Pin
- added J2: Conn_01x03_Pin, Connector_PinHeader_2.54mm:PinHeader_1x03_P2.54mm_Vertical, symbol Connector:Conn_01x03_Pin
Connections:
- net GND: now also J1.2 (Pin_2), J2.1 (Pin_1)
- net VCC: now also J2.3 (Pin_3)
- net at C1.2, RV1.2, U1.17 (GP26): now also J2.2 (Pin_2)
- net at R1.2, S1.2, U1.3 (GP2): now also J1.1 (Pin_1)
Other:
- moved on the sheet: C1, RV1
