File: usbPaddleSingleKicad/usbPaddleSingleKicad.kicad_pcb (KiCad board)
At the start: 2 copper layers, 90 x 43 mm, 17 parts, among them U1 RP2040-ZERO, U2 RJ116P4C, U3 RJ116P4C, U4 RJ116P4C, U5 RJ116P4C

Commit message: new single paddle pcb
Parts:
- removed the ? at (95.6, 95.0)
- removed the ? at (177.6, 95.0)
- removed the ? at (95.6, 60.0)
- removed the ? at (177.6, 60.0)
- removed C2, C3, C4: .1µF, Capacitor_THT:C_Disc_D3.8mm_W2.6mm_P2.50mm
- removed R2, R3, R4: 10kΩ, Resistor_THT:R_Axial_DIN0309_L9.0mm_D3.2mm_P12.70mm_Horizontal
- removed U2, U3, U4, U5: RJ116P4C, RJ116P4C:RJ6P4C_GLX-N-64M
- added ?: , , F.Cu at (156.6, 43.5)
- added ?: , , F.Cu at (116.6, 43.5)
- added ?: , , F.Cu at (121.1, 106.5)
- added ?: , , F.Cu at (152.1, 106.5)
- added J1: Conn_01x02_Pin, Connector_PinHeader_2.54mm:PinHeader_1x02_P2.54mm_Vertical, F.Cu at (122.1, 66.7)
- added RV1: R_Potentiometer, Potentiometer_THT:Potentiometer_Alps_RK09K_Single_Vertical, F.Cu at (139.1, 86.9)
- added S1: ~, Button_Switch_Keyboard:SW_Cherry_MX_1.00u_Plate, F.Cu at (125.2, 50.2)
- moved U1 18.9 mm to (143.9, 50.5)
- moved C1 18.0 mm to (139.1, 83.4), turned to 180 degrees
- moved R1 11.8 mm to (157.4, 61.3), turned to 90 degrees
Connections:
- R1 pad 2: Net-(U1-GP1) -> Net-(J1-Pin_1)
- U1 pad 18: Net-(U1-GP27) -> unconnected-(U1-GP27-Pad18)
- U1 pad 19: Net-(U1-GP28) -> unconnected-(U1-GP28-Pad19)
- U1 pad 2: Net-(U1-GP1) -> unconnected-(U1-GP1-Pad2)
- U1 pad 20: Net-(U1-GP29) -> unconnected-(U1-GP29-Pad20)
- U1 pad 3: Net-(U1-GP2) -> Net-(J1-Pin_1)
- U1 pad 8: Net-(U1-GP7) -> unconnected-(U1-GP7-Pad8)
- U1 pad 9: Net-(U1-GP8) -> unconnected-(U1-GP8-Pad9)
Routing:
- net VCC: track 196.7 -> 91.9 mm, vias 2 -> 0
- net Net-(U1-GP2): track 67.8 -> 0.00 mm
- net Net-(J1-Pin_1): track 0.00 -> 59.6 mm
- net Net-(U1-GP29): track 49.8 -> 0.00 mm
- net Net-(U1-GP1): track 45.8 -> 0.00 mm
- net Net-(U1-GP7): track 39.3 -> 0.00 mm
- net Net-(U1-GP28): track 32.8 -> 0.00 mm
- net Net-(U1-GP27): track 27.5 -> 0.00 mm
- net Net-(U1-GP8): track 24.9 -> 0.00 mm
- net Net-(J2-Pin_2): track 42.8 -> 32.1 mm
- net GND: vias 34 -> 6
Other:
- board size 90 x 43 mm -> 51 x 72.5 mm
- board text added: "USB Paddle version 1.0 Dan Shimmyo May 2026"
- board text removed: "BTN"
- board text removed: "P1"
- board text removed: "P2"
- board text removed: "P3"
- board text removed: "P4"
- board text removed: "Paddle Controller Base Unit version 1.0 Dan Shimmyo May 2026"

Commit message: adjust layout
Parts:
- moved R1 20.7 mm to (137.5, 67.2), turned to 0 degrees
Routing:
- net Net-(J1-Pin_1): track 59.6 -> 76.4 mm
- net VCC: track 91.9 -> 88.7 mm
- net Net-(J2-Pin_2): track 32.1 -> 34.4 mm
- net GND: vias 6 -> 11
Changed lines of the file:
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@@
 	(footprint "Resistor_THT:R_Axial_DIN0309_L9.0mm_D3.2mm_P12.70mm_Horizontal"
 		(layer "F.Cu")
-		(at 157.395 61.325 90)
+		(at 137.545 67.225)
 		(descr "Resistor, Axial_DIN0309 series, Axial, Horizontal, pin pitch=12.7mm, 0.5W = 1/2W, length*diameter=9*3.2mm^2, http://cdn-reichelt.de/documents/datenblatt/B400/1_4W%23YAG.pdf")
 		(tags "Resistor Axial_DIN0309 series Axial Horizontal pin pitch 12.7mm 0.5W = 1/2W length 9mm diameter 3.2mm")
 		(property "Reference" "R1"
-			(at 6.35 -2.72 90)
+			(at 6.35 -2.72 0)
 			(layer "F.SilkS")
 			(effects
@@
 		)
 		(property "Value" "10kΩ"
-			(at 6.35 2.72 90)
+			(at 6.35 2.72 0)
 			(layer "F.Fab")
 			(effects
@@
 		)
 		(property "Datasheet" ""
-			(at 0 0 90)
+			(at 0 0 0)
 			(layer "F.Fab")
 			(hide yes)
@@
 		)
 		(property "Description" "Resistor"
-			(at 0 0 90)
+			(at 0 0 0)
 			(layer "F.Fab")
 			(hide yes)
@@
 		)
 		(property "KiLib_Generator" "resistor/THT"
-			(at 0 0 90)
+			(at 0 0 0)
 			(layer "F.SilkS")
 			(hide yes)
@@
 		(duplicate_pad_numbers_are_jumpers no)
 		(fp_line
+			(start 1.04 0)
+			(end 1.73 0)
+			(stroke
+				(width 0.12)
+				(type solid)
+			)
+			(layer "F.SilkS")
+		)
+		(fp_line
 			(start 11.66 0)
 			(end 10.97 0)
-			(stroke
-				(width 0.12)
-				(type solid)
-			)
-			(layer "F.SilkS")
-		)
-		(fp_line
-			(start 1.04 0)
-			(end 1.73 0)
 			(stroke
 				(width 0.12)
@@
 		)
 		(fp_line
+			(start 0 0)
+			(end 1.85 0)
+			(stroke
+				(width 0.1)
+				(type solid)
+			)
+			(layer "F.Fab")
+		)
+		(fp_line
 			(start 12.7 0)
 			(end 10.85 0)
-			(stroke
-				(width 0.1)
-				(type solid)
-			)
-			(layer "F.Fab")
-		)
-		(fp_line
-			(start 0 0)
-			(end 1.85 0)
 			(stroke
 				(width 0.1)
@@
 		)
 		(fp_text user "${REFERENCE}"
-			(at 6.35 0 90)
+			(at 6.35 0 0)
 			(layer "F.Fab")
 			(effects
@@
 		)
 		(pad "1" thru_hole circle
-			(at 0 0 90)
+			(at 0 0)
 			(size 1.6 1.6)
 			(drill 0.8)
@@
 		)
 		(pad "2" thru_hole circle
-			(at 12.7 0 90)
+			(at 12.7 0)
 			(size 1.6 1.6)
 			(drill 0.8)
@@
 	)
 	(via
-		(at 126.395 52.975)
+		(at 139.145 44.475)
+		(size 0.6)
+		(drill 0.3)
+		(layers "F.Cu" "B.Cu")
+		(free yes)
+		(net "GND")
+	)
+	(via
+		(at 127.895 52.475)
 		(size 0.6)
 		(drill 0.3)
@@
 		)
 		(filling no)
+		(net "GND")
+	)
+	(via
+		(at 138.895 41.975)
+		(size 0.6)
+		(drill 0.3)
+		(layers "F.Cu" "B.Cu")
+		(free yes)
+		(net "GND")
+	)
+	(via
+		(at 125.145 60.725)
+		(size 0.6)
+		(drill 0.3)
+		(layers "F.Cu" "B.Cu")
+		(free yes)
 		(net "GND")
 	)
@@
 		(net "GND")
 	)
+	(via
+		(at 128.645 66.725)
+		(size 0.6)
+		(drill 0.3)
+		(layers "F.Cu" "B.Cu")
+		(free yes)
+		(net "GND")
+	)
+	(via
+		(at 133.895 41.225)
+		(size 0.6)
+		(drill 0.3)
+		(layers "F.Cu" "B.Cu")
+		(free yes)
+		(net "GND")
+	)
 	(segment
 		(start 136.645 86.925)
@@
 	)
 	(segment
-		(start 137.329 56.609)
-		(end 136.275 55.555)
+		(start 133.645 56.975)
+		(end 135.065 55.555)
 		(width 0.2)
 		(layer "F.Cu")
@@
 	)
 	(segment
-		(start 137.329 64.166)
-		(end 137.329 56.609)
+		(start 136.595 83.375)
+		(end 133.645 80.425)
 		(width 0.2)
 		(layer "F.Cu")
@@
 	)
 	(segment
-		(start 136.595 64.9)
-		(end 137.329 64.166)
+		(start 135.065 55.555)
+		(end 136.275 55.555)
 		(width 0.2)
 		(layer "F.Cu")
@@
 	)
 	(segment
-		(start 136.595 83.375)
-		(end 136.595 64.9)
+		(start 133.645 80.425)
+		(end 133.645 56.975)
 		(width 0.2)
 		(layer "F.Cu")
@@
 	)
 	(segment
-		(start 147.605 56.725)
-		(end 152.795 56.725)
+		(start 133.645 48.025)
+		(end 133.645 63.325)
+		(width 0.4)
+		(layer "B.Cu")
+		(net "VCC")
+	)
+	(segment
+		(start 133.645 63.325)
+		(end 137.545 67.225)
 		(width 0.4)
 		(layer "B.Cu")
@@
 	)
 	(segment
-		(start 152.795 56.725)
-		(end 157.395 61.325)
-		(width 0.4)
-		(layer "B.Cu")
-		(net "VCC")
-	)
-	(segment
 		(start 136.275 45.395)
-		(end 147.605 56.725)
+		(end 133.645 48.025)
 		(width 0.4)
 		(layer "B.Cu")
@@
 	)
 	(segment
-		(start 124.995 54.301598)
-		(end 123.428402 52.735)
+		(start 151.515 45.395)
+		(end 152.569 46.449)
 		(width 0.2)
 		(layer "F.Cu")
@@
 	)
 	(segment
-		(start 156.045 48.625)
-		(end 152.815 45.395)
+		(start 148.994418 67.225)
+		(end 150.245 67.225)
+		(width 0.2)
+		(layer "F.Cu")
+		(net "Net-(J1-Pin_1)")
+	)
+	(segment
+		(start 142.409 60.198418)
+		(end 142.409 60.639582)
 		(width 0.2)
 		(layer "F.Cu")
@@
 	)
 	(segment
-		(start 123.428402 52.735)
-		(end 118.835 52.735)
+		(start 152.569 64.901)
+		(end 150.245 67.225)
+		(width 0.2)
+		(layer "F.Cu")
+		(net "Net-(J1-Pin_1)")
+	)
+	(segment
+		(start 142.409 60.639582)
+		(end 148.994418 67.225)
 		(width 0.2)
 		(layer "F.Cu")
@@
 	)
 	(segment
-		(start 157.395 48.625)
-		(end 156.045 48.625)
+		(start 136.711582 54.501)
+		(end 142.409 60.198418)
 		(width 0.2)
 		(layer "F.Cu")
@@
 	)
 	(segment
-		(start 152.815 45.395)
-		(end 151.515 45.395)
+		(start 118.835 52.735)
+		(end 124.905 52.735)
 		(width 0.2)
 		(layer "F.Cu")
@@
 	)
 	(segment
-		(start 151.515 45.395)
-		(end 142.608402 54.301598)
+		(start 124.905 52.735)
+		(end 126.671 54.501)
 		(width 0.2)
 		(layer "F.Cu")
@@
 	)
 	(segment
-		(start 142.608402 54.301598)
-		(end 124.995 54.301598)
+		(start 152.569 46.449)
+		(end 152.569 64.901)
 		(width 0.2)
 		(layer "F.Cu")
 		(net "Net-(J1-Pin_1)")
 	)
+	(segment
+		(start 126.671 54.501)
+		(end 136.711582 54.501)
+		(width 0.2)
+		(layer "F.Cu")
+		(net "Net-(J1-Pin_1)")
+	)
+	(segment
+		(start 150.129 67.109)
+		(end 150.245 67.225)
+		(width 0.4)
+		(layer "B.Cu")
+		(net "Net-(J1-Pin_1)")
+	)
